File: Internal_Breakout/Internal_Breakout.brd (EAGLE design)
At the start: 38.5 x 27.5 mm, 31 parts, among them T1 2N4401, T2 2N4401, U1 MCP10804-T, U2 MIC5205-5V

Commit message: Licenses
Parts:
- added D1: FM4007W, CYCFI_diode:SMX
- added H5, H6: (no value), con-lstb:MA03-1_
- moved H10 2.50 mm to (30.9, 21.7)
- moved H11 2.50 mm to (33.6, 21.7)
- moved H12 2.50 mm to (36.3, 21.7)
- moved H13 2.50 mm to (30.9, 12.3)
- moved H14 2.50 mm to (33.6, 12.3)
- moved H15 2.50 mm to (36.3, 12.3)
- moved H9 2.50 mm to (28.2, 21.7)
Connections:
- new net N$4: C12.1, C6.1, D1.CATHODE, U1.3, U2.1, U2.3
- net 5.4V: now also H5.2, H6.2
- net 9.3V: now also H5.3, H6.3
- net GND: now also H5.1, H6.1
- net VCC: now also D1.ANODE; no longer C12.1, C6.1, U1.3, U2.1, U2.3
Routing:
- net GND: track 110.8 -> 140.6 mm, vias 2 -> 7
- net N$4: track 0.00 -> 27.3 mm, vias 0 -> 4
- net 5.4V: track 47.6 -> 68.6 mm, vias 3 -> 5
- net 9.3V: track 42.7 -> 48.3 mm
- net CH11: track 51.1 -> 53.5 mm, vias 2 -> 3
- net CH10: track 44.9 -> 47.4 mm
- net MIDI3: track 38.4 -> 40.9 mm
- net MIDI2: track 29.4 -> 31.6 mm
- net MIDI1: track 29.1 -> 31.1 mm
- net CH12: track 50.6 -> 52.3 mm, vias 2 -> 3
- net VCC: track 36.6 -> 38.2 mm, vias 4 -> 0
- net CH9: track 44.5 -> 45.7 mm
Other:
- board size 38.5 x 27.5 mm -> 41 x 27.5 mm
- board text added: "5V"
- board text added: "D1"
- board text added: "v1.2"
- board text removed: "v1.1"
