File: Internal_Breakout/Internal_Breakout.kicad_pcb (KiCad board)
At the start: 2 copper layers, 50 x 35 mm, 22 parts, among them J1 CONN_01X03, J10 CONN_01X10, J11 CONN_01X10, J12 CONN_01X03, J13 CONN_01X03, J2 CONN_01X03, J3 CONN_01X10, J4 CONN_01X10, J5 CONN_01X03, J6 CONN_01X03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

Commit message: Updated Internal Breakout Files
Parts:
- C1, C3, C5, C6: footprint Capacitors_SMD:C_0603 -> Capacitors_SMD:C_0603_HandSoldering
- moved J5 5.06 mm to (159.8, 49.2), turned to 270 degrees
- moved J6 5.05 mm to (159.8, 45.5), turned to 270 degrees
- moved J1 5.05 mm to (148.9, 45.5), turned to 270 degrees
- moved J7 5.05 mm to (172.7, 49.2), turned to 270 degrees
- moved J2 5.05 mm to (148.9, 49.2), turned to 270 degrees
- moved J8 5.04 mm to (172.6, 45.5), turned to 270 degrees
- moved J9 5.04 mm to (172.6, 52.9), turned to 270 degrees
- moved Q1 4.71 mm to (153.8, 62.8)
- moved C4 4.52 mm to (150.0, 62.2)
- moved C1 4.41 mm to (158.4, 57.5)
- moved U1 4.14 mm to (153.8, 57.5)
- moved C2 3.47 mm to (154.7, 54.6)
- moved C3 1.97 mm to (150.1, 57.4)
- moved C5 0.98 mm to (147.5, 57.4)
- moved J13 0.90 mm to (168.8, 57.6)
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Connections:
- J10 pad 10: CH10 -> GND
- J11 pad 1: CH11 -> CH10
- J11 pad 2: CH12 -> CH11
- J11 pad 3: CH13 -> CH12
- J11 pad 4: CH14 -> CH13
- J11 pad 5: CH15 -> CH14
- J11 pad 6: +15V_REG -> CH15
- J11 pad 7: +15V_REG -> +VDC_IN
- J11 pad 8: GND -> +VDC_IN
- Q1 pad 3: +15V_REG -> +VDC_IN
Routing:
- net +VDC_IN: track 0.00 -> 12.3 mm
- net +15V_REG: track 10.00 -> 0.00 mm
- net CH11: track 60.0 -> 69.3 mm
- net CH14: track 89.7 -> 82.3 mm, vias 1 -> 2
- net CH13: track 87.8 -> 80.7 mm
- net CH9: track 59.6 -> 64.0 mm
- net CH12: track 59.4 -> 62.3 mm
- net +10VA: track 135.6 -> 133.1 mm
- net CH15: track 77.4 -> 79.3 mm, vias 2 -> 1
- net Net-(C1-Pad1): track 13.4 -> 11.7 mm
- net Net-(C2-Pad1): track 3.95 -> 3.04 mm
Other:
- board text added: "CH9 - CH15"
- board text removed: "CH9 - CH12"
