File: Internal_Breakout/Internal_Breakout.sch (KiCad schematic (older format))
At the start: 21 parts, among them J1 CONN_01X03, J10 CONN_01X10, J11 CONN_01X10, J12 CONN_01X03, J13 CONN_01X03, J2 CONN_01X03, J3 CONN_01X10, J4 CONN_01X10, J5 CONN_01X03, J6 CONN_01X03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

Commit message: Updated Internal Breakout Files
Parts:
- C1, C3, C5, C6: footprint Capacitors_SMD:C_0603 -> Capacitors_SMD:C_0603_HandSoldering
