File: Nu_Capsule/Nu_Capsule.sch (EAGLE design)
At the start: 20 parts, among them T1 2SC3324, T2 2SC3324

Commit message: Doc updates
Parts:
- C5: value 1uF -> 4.7uF
- R6: value 47K -> 10K
Other:
- moved on the sheet: C1, C2, C3, C4, C5, H1, H2, R1, R2, R3, R4, R5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

Commit message: updates and minor corrections
Parts:
- C5: value 4.7uF -> 1uF
- R6: value 10K -> 47K
Other:
- moved on the sheet: C1, C2, C3, C4, C5, H1, H2, R1, R2, R3, R4, R5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

Commit message: more updates; tweaks
Parts:
- C5: value 1uF -> 4.7uF
- R6: value 47K -> 10K
Other:
- moved on the sheet: C1, C2, C3, C4, C5, H1, H2, R1, R2, R3, R4, R5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

Commit message: Licenses
Parts:
- C1, C5: device resistor:C-EUC0805 -> resistor:C-EUC0603
- R2: device resistor:R-EU_R0805 -> resistor:R-EU_R0402
Other:
- note added: "Nu Preamp Project by Cycfi Research is licensed under a Creative Commons Attribution-ShareAlike 4.0 International License. Copyright CYCFI Research Inc. 2013-2016"
- note removed: "Nu Project by Cycfi Research is licensed under a Creative Commons Attribution-NonCommercial 4.0 International License. http://creativecommons.org/licenses/by-nc/4.0/ Copyright CYCFI Research Inc. 2013-2016"
- moved on the sheet: C1, C2, C3, C4, C5, H1, H2, R1, R2, R3, R4, R5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

Commit message: *update license date
Other:
- note added: "201719"
- note added: "Nu Preamp Project by Cycfi Research is licensed under a Creative Commons Attribution-ShareAlike 4.0 International License. Copyright CYCFI Research Inc. 2013-2017"
- note removed: "2016035"
- note removed: "Nu Preamp Project by Cycfi Research is licensed under a Creative Commons Attribution-ShareAlike 4.0 International License. Copyright CYCFI Research Inc. 2013-2016"
Changed lines of the file:
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@@
 <text x="12.7" y="12.7" size="2.54" layer="95">Nu Preamp Project by Cycfi Research is licensed under a
 Creative Commons Attribution-ShareAlike 4.0 International License.
-Copyright CYCFI Research Inc. 2013-2016</text>
+Copyright CYCFI Research Inc. 2013-2017</text>
 <text x="73.66" y="77.47" size="1.778" layer="95">NC: SMD pads used
 for coil soldering</text>
@@
 <wire x1="90.17" y1="86.995" x2="79.375" y2="86.995" width="0.1524" layer="94"/>
 <wire x1="79.375" y1="86.995" x2="79.375" y2="88.265" width="0.1524" layer="94"/>
-<text x="200.66" y="11.43" size="2.54" layer="95">2016035</text>
+<text x="200.66" y="11.43" size="2.54" layer="95">201719</text>
 <text x="92.71" y="88.9" size="1.778" layer="95">OC</text>
 <text x="92.71" y="95.885" size="1.778" layer="95">IC</text>
