File: Nu_Capsule/Nu_Preamp.sch (EAGLE design)
At the start: 27 parts, among them Q1 2SC3324, Q2 2SC3324, U1 TLV170

Commit message: push updated Nu preamp schematic files
Other:
- note added: "Nu Project by Cycfi Research is licensed under a Creative Commons Attribution-ShareAlike 4.0 International License. http://creativecommons.org/licenses/by-nc/4.0/ Copyright CYCFI Research Inc. 2013-2019"
- note added: "U1"
- note removed: "Nu Project by Cycfi Research is licensed under a Creative Commons Attribution-ShareAlike 4.0 International License. http://creativecommons.org/licenses/by-nc/4.0/ Copyright CYCFI Research Inc. 2013-2018"
