File: GK_Roland_Breakout/GK_Roland_Breakout.sch (EAGLE design)
At the start: 39 parts, among them T2 2N4401, U1 RC4558, U2 MIC5205-5V

Commit message: *update license date
Other:
- note added: "201722"
- note added: "GK Roland Breakout Project by Cycfi Research is licensed under a Creative Commons Attribution-ShareAlike 4.0 International License. Copyright CYCFI Research Inc. 2013-2017"
- note removed: "GK Roland Breakout by Cycfi Research is licensed under a Creative Commons Attribution-NonCommercial 4.0 International License. http://creativecommons.org/licenses/by-nc/4.0/ Copyright CYCFI Research Inc. 2013-2016"
Changed lines of the file:
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@@
 <setting verticaltext="up"/>
 </settings>
-<grid distance="0.05" unitdist="inch" unit="inch" style="lines" multiple="1" display="yes" altdistance="0.01" altunitdist="inch" altunit="inch"/>
+<grid distance="0.1" unitdist="inch" unit="inch" style="lines" multiple="1" display="no" altdistance="0.01" altunitdist="inch" altunit="inch"/>
 <layers>
 <layer number="1" name="Top" color="4" fill="1" visible="no" active="no"/>
@@
 <sheet>
 <plain>
-<text x="13.97" y="8.89" size="2.54" layer="95">GK Roland Breakout by Cycfi Research is licensed under a
-Creative Commons Attribution-NonCommercial 4.0
-International License.
-http://creativecommons.org/licenses/by-nc/4.0/
-Copyright CYCFI Research Inc. 2013-2016</text>
+<text x="13.97" y="8.89" size="2.54" layer="95">GK Roland Breakout Project by Cycfi Research is licensed under a
+Creative Commons Attribution-ShareAlike 4.0 International License.
+Copyright CYCFI Research Inc. 2013-2017</text>
 <text x="162.56" y="19.05" size="2.54" layer="95">Internal Breakout Board - GK</text>
 <wire x1="178.362721875" y1="25.186403125" x2="163.27975" y2="25.186403125" width="0" layer="94"/>
@@
 <text x="33.655" y="71.755" size="1.778" layer="95" rot="R180">GND</text>
 <text x="236.22" y="7.62" size="2.54" layer="95">0.9</text>
+<text x="185.42" y="11.43" size="2.54" layer="95">201722</text>
 </plain>
 <instances>
