File: internal_breakout/internal_breakout.sch (EAGLE design)
At the start: 21 parts, among them J10 2X5, J11 2X5, J3 2X5, J4 2X5, Q1 DMP3099L, U1 LP2985

Commit message: push updated files for internal breakout
Parts:
- added FB1: BLM18KG700TN1D, SamacSys_Parts:BLM18KG700TN1D
- added J14, J15, J16: (no value), con-lstb:MA03-1
- C1: value 1uF -> 10uF; SPICEPREFIX (none) -> C
Connections:
- removed net NC: J4.2
- new net +10VA: C2.1, C3.1, C5.1, C6.1, J12.3, J14.3, U1.VOUT
- new net VIN: J11.7, J11.8, Q1.D
- net CH10: now also J4.6; no longer J4.8
- net CH11: now also J4.3; no longer J4.5
- net CH12: now also J4.4; no longer J4.6
- net CH13: now also J4.1; no longer J4.3
- net CH14: now also J4.2; no longer J4.4
- net CH15: no longer J4.1
- net CH7: now also J15.3, J4.7
- net CH8: now also J16.3, J4.8
- net CH9: now also J4.5; no longer J4.7
- net GND: now also J15.2, J16.2
- net N$1: now also FB1.1; no longer C1.1, U1.ON/OFF, U1.VIN
- net V+: now also J14.2, J15.1, J16.1; no longer C2.1, C3.1, C5.1, C6.1, J12.3, J13.3, U1.VOUT
- net VCC: now also C1.1, FB1.2, J13.3, J14.1, U1.ON/OFF, U1.VIN; no longer J11.7, J11.8, Q1.D
Other:
- note added: "AUDIO / CV INPUTS (CH9 - CH15)"
- note added: "Internal Breakout Project by Cycfi Research is licensed under a Creative Commons Attribution-ShareAlike 4.0 International License. Copyright CYCFI Research Inc. 2013-2020"
- note added: "POWER SELECT REGULATED/ UNREGULATED"
- note added: "v2.2"
- note removed: "+10VA"
- note removed: "201706282"
- note removed: "CH10"
- note removed: "CH11"
- note removed: "CH12"
- note removed: "CH13"
- note removed: "CH14"
- note removed: "CH15"
- note removed: "CH9"
- note removed: "CV INPUTS (CH13 - CH15)"
- note removed: "EXTERNAL PICKUPS (CH9 - CH12)"
- note removed: "Internal Breakout Project by Cycfi Research is licensed under a Creative Commons Attribution-ShareAlike 4.0 International License. Copyright CYCFI Research Inc. 2013-2019"
- note removed: "NC"
- note removed: "POWER SUPPLY"
- note removed: "v2.0"
- moved on the sheet: C1, C2, C3, C4, C5, C6, J1, J10, J11, J2, J3, J4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

Commit message: update internal breakout files
Other:
- note added: "v2.5"
- note removed: "v2.2"
Changed lines of the file:
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@@
 <plain>
 <text x="195.58" y="19.05" size="2.54" layer="95" font="vector">Internal Breakout</text>
-<text x="254" y="6.985" size="2.1844" layer="95" font="vector">v2.2</text>
+<text x="254" y="6.985" size="2.1844" layer="95" font="vector">v2.5</text>
 <text x="7.62" y="7.62" size="2.1844" layer="95" font="vector">Internal Breakout Project by Cycfi Research is licensed under a
 Creative Commons Attribution-ShareAlike 4.0 International License.

Commit message: update internal breakout with special header for 2 way switch
Parts:
- added J17: (no value), con-lstb:MA03-1
Connections:
- net CH7: now also J17.3
- net CH8: now also J17.1
- net GND: now also J17.2
Other:
- note added: "2 WAY SWITCH CONNECTOR"
Changed lines of the file:
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@@
 <setting verticaltext="up"/>
 </settings>
-<grid distance="0.1" unitdist="inch" unit="inch" style="lines" multiple="1" display="no" altdistance="0.01" altunitdist="inch" altunit="inch"/>
+<grid distance="0.025" unitdist="inch" unit="inch" style="lines" multiple="1" display="yes" altdistance="0.01" altunitdist="inch" altunit="inch"/>
 <layers>
 <layer number="1" name="Top" color="4" fill="1" visible="no" active="no"/>
@@
 </part>
 <part name="J16" library="con-lstb" deviceset="MA03-1" device="">
+<attribute name="MF" value=""/>
+<attribute name="MPN" value=""/>
+<attribute name="OC_FARNELL" value="unknown"/>
+<attribute name="OC_NEWARK" value="unknown"/>
+</part>
+<part name="J17" library="con-lstb" deviceset="MA03-1" device="">
 <attribute name="MF" value=""/>
 <attribute name="MPN" value=""/>
@@
 <rectangle x1="214.78875" y1="31.90875" x2="222.91675" y2="31.97225" layer="95"/>
 <rectangle x1="223.48825" y1="31.90875" x2="225.83775" y2="31.97225" layer="95"/>
+<text x="108.585" y="85.725" size="1.778" layer="95" rot="R90">2 WAY SWITCH
+  CONNECTOR</text>
 </plain>
 <instances>
@@
 <instance part="J15" gate="G$1" x="115.57" y="71.12"/>
 <instance part="J16" gate="G$1" x="115.57" y="55.88"/>
+<instance part="J17" gate="G$1" x="115.57" y="95.885"/>
 </instances>
 <busses>
@@
 <label x="127" y="55.245" size="1.778" layer="95"/>
 </segment>
+<segment>
+<pinref part="J17" gate="G$1" pin="2"/>
+<wire x1="123.19" y1="95.885" x2="125.73" y2="95.885" width="0.1524" layer="91"/>
+<label x="132.715" y="96.52" size="1.778" layer="95" rot="R180"/>
+</segment>
 </net>
 <net name="VIN" class="0">
@@
 <label x="127" y="73.025" size="1.778" layer="95"/>
 </segment>
+<segment>
+<pinref part="J17" gate="G$1" pin="3"/>
+<wire x1="123.19" y1="98.425" x2="125.73" y2="98.425" width="0.1524" layer="91"/>
+<label x="132.08" y="99.695" size="1.778" layer="95" rot="R180"/>
+</segment>
 </net>
 <net name="CH2" class="0">
@@
 <label x="127" y="57.785" size="1.778" layer="95"/>
 </segment>
+<segment>
+<pinref part="J17" gate="G$1" pin="1"/>
+<wire x1="123.19" y1="93.345" x2="125.73" y2="93.345" width="0.1524" layer="91"/>
+<label x="132.08" y="93.98" size="1.778" layer="95" rot="R180"/>
+</segment>
 </net>

Commit message: Update fix: Audio/CV now starts at CH7
Other:
- note added: "AUDIO / CV INPUTS (CH7 - CH15)"
- note removed: "AUDIO / CV INPUTS (CH9 - CH15)"
Changed lines of the file:
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@@
 <?xml version="1.0" encoding="utf-8"?>
 <!DOCTYPE eagle SYSTEM "eagle.dtd">
-<eagle version="6.3">
+<eagle version="9.6.1">
 <drawing>
 <settings>
 <setting alwaysvectorfont="no"/>
+<setting keepoldvectorfont="yes"/>
 <setting verticaltext="up"/>
 </settings>
-<grid distance="0.025" unitdist="inch" unit="inch" style="lines" multiple="1" display="yes" altdistance="0.01" altunitdist="inch" altunit="inch"/>
+<grid distance="0.1" unitdist="inch" unit="inch" style="lines" multiple="1" display="no" altdistance="0.01" altunitdist="inch" altunit="inch"/>
 <layers>
 <layer number="1" name="Top" color="4" fill="1" visible="no" active="no"/>
@@
 <text x="25.4" y="106.68" size="1.778" layer="95" rot="R90">FROM NU MULTI</text>
 <text x="106.68" y="63.5" size="1.778" layer="95" rot="R90" align="center">AUDIO / CV INPUTS
-   (CH9 - CH15)</text>
+   (CH7 - CH15)</text>
 <text x="25.4" y="35.56" size="1.778" layer="95" rot="R90" align="center">SUPPLY
 EXTENSIONS</text>
@@
 </plain>
 <instances>
-<instance part="FRAME2" gate="G$1" x="0" y="0"/>
+<instance part="FRAME2" gate="G$1" x="0" y="0" smashed="yes"/>
 <instance part="FRAME2" gate="G$2" x="162.56" y="0" smashed="yes">
 <attribute name="SHEET" x="248.92" y="1.27" size="2.54" layer="94" font="vector"/>
@@
 <attribute name="NAME" x="132.334" y="163.068" size="1.778" layer="95"/>
 </instance>
-<instance part="C2" gate="G$1" x="162.56" y="154.94"/>
-<instance part="C3" gate="G$1" x="170.18" y="154.94"/>
-<instance part="C4" gate="G$1" x="154.94" y="144.78"/>
-<instance part="C5" gate="G$1" x="177.8" y="154.94"/>
-<instance part="SUPPLY1" gate="GND" x="139.7" y="134.62"/>
+<instance part="C2" gate="G$1" x="162.56" y="154.94" smashed="yes">
+<attribute name="NAME" x="164.084" y="155.321" size="1.778" layer="95"/>
+<attribute name="VALUE" x="164.084" y="150.241" size="1.778" layer="96"/>
+</instance>
+<instance part="C3" gate="G$1" x="170.18" y="154.94" smashed="yes">
+<attribute name="NAME" x="171.704" y="155.321" size="1.778" layer="95"/>
+<attribute name="VALUE" x="171.704" y="150.241" size="1.778" layer="96"/>
+</instance>
+<instance part="C4" gate="G$1" x="154.94" y="144.78" smashed="yes">
+<attribute name="NAME" x="156.464" y="145.161" size="1.778" layer="95"/>
+<attribute name="VALUE" x="156.464" y="140.081" size="1.778" layer="96"/>
+</instance>
+<instance part="C5" gate="G$1" x="177.8" y="154.94" smashed="yes">
+<attribute name="NAME" x="179.324" y="155.321" size="1.778" layer="95"/>
+<attribute name="VALUE" x="179.324" y="150.241" size="1.778" layer="96"/>
+</instance>
+<instance part="SUPPLY1" gate="GND" x="139.7" y="134.62" smashed="yes">
+<attribute name="VALUE" x="137.795" y="131.445" size="1.778" layer="96"/>
+</instance>
 <instance part="J3" gate="G$1" x="50.8" y="127" smashed="yes">
 <attribute name="NAME" x="45.72" y="135.255" size="1.27" layer="95" font="vector"/>
@@
 <attribute name="NAME" x="220.98" y="112.395" size="1.27" layer="95" font="vector"/>
 </instance>
-<instance part="C6" gate="G$1" x="185.42" y="154.94"/>
-<instance part="J1" gate="G$1" x="135.89" y="71.12"/>
-<instance part="J2" gate="G$1" x="135.89" y="55.88"/>
-<instance part="J13" gate="G$1" x="48.26" y="33.02"/>
-<instance part="J6" gate="G$1" x="163.83" y="71.12"/>
-<instance part="J5" gate="G$1" x="163.83" y="55.88"/>
-<instance part="J12" gate="G$1" x="96.52" y="33.02"/>
-<instance part="J8" gate="G$1" x="194.31" y="71.12"/>
-<instance part="J7" gate="G$1" x="194.31" y="55.88"/>
-<instance part="J9" gate="G$1" x="223.52" y="71.12"/>
-<instance part="J14" gate="G$1" x="48.26" y="60.96"/>
-<instance part="C1" gate="G$1" x="111.76" y="154.94"/>
+<instance part="C6" gate="G$1" x="185.42" y="154.94" smashed="yes">
+<attribute name="NAME" x="186.944" y="155.321" size="1.778" layer="95"/>
+<attribute name="VALUE" x="186.944" y="150.241" size="1.778" layer="96"/>
+</instance>
+<instance part="J1" gate="G$1" x="135.89" y="71.12" smashed="yes">
+<attribute name="VALUE" x="134.62" y="63.5" size="1.778" layer="96"/>
+<attribute name="NAME" x="134.62" y="76.962" size="1.778" layer="95"/>
+</instance>
+<instance part="J2" gate="G$1" x="135.89" y="55.88" smashed="yes">
+<attribute name="VALUE" x="134.62" y="48.26" size="1.778" layer="96"/>
+<attribute name="NAME" x="134.62" y="61.722" size="1.778" layer="95"/>
+</instance>
+<instance part="J13" gate="G$1" x="48.26" y="33.02" smashed="yes">
+<attribute name="VALUE" x="46.99" y="25.4" size="1.778" layer="96"/>
+<attribute name="NAME" x="46.99" y="38.862" size="1.778" layer="95"/>
+</instance>
+<instance part="J6" gate="G$1" x="163.83" y="71.12" smashed="yes">
+<attribute name="VALUE" x="162.56" y="63.5" size="1.778" layer="96"/>
+<attribute name="NAME" x="162.56" y="76.962" size="1.778" layer="95"/>
+</instance>
+<instance part="J5" gate="G$1" x="163.83" y="55.88" smashed="yes">
+<attribute name="VALUE" x="162.56" y="48.26" size="1.778" layer="96"/>
+<attribute name="NAME" x="162.56" y="61.722" size="1.778" layer="95"/>
+</instance>
+<instance part="J12" gate="G$1" x="96.52" y="33.02" smashed="yes">
+<attribute name="VALUE" x="95.25" y="25.4" size="1.778" layer="96"/>
+<attribute name="NAME" x="95.25" y="38.862" size="1.778" layer="95"/>
+</instance>
+<instance part="J8" gate="G$1" x="194.31" y="71.12" smashed="yes">
+<attribute name="VALUE" x="193.04" y="63.5" size="1.778" layer="96"/>
+<attribute name="NAME" x="193.04" y="76.962" size="1.778" layer="95"/>
+</instance>
+<instance part="J7" gate="G$1" x="194.31" y="55.88" smashed="yes">
+<attribute name="VALUE" x="193.04" y="48.26" size="1.778" layer="96"/>
+<attribute name="NAME" x="193.04" y="61.722" size="1.778" layer="95"/>
+</instance>
+<instance part="J9" gate="G$1" x="223.52" y="71.12" smashed="yes">
+<attribute name="VALUE" x="222.25" y="63.5" size="1.778" layer="96"/>
+<attribute name="NAME" x="222.25" y="76.962" size="1.778" layer="95"/>
+</instance>
+<instance part="J14" gate="G$1" x="48.26" y="60.96" smashed="yes">
+<attribute name="VALUE" x="46.99" y="53.34" size="1.778" layer="96"/>
+<attribute name="NAME" x="46.99" y="66.802" size="1.778" layer="95"/>
+</instance>
+<instance part="C1" gate="G$1" x="111.76" y="154.94" smashed="yes">
+<attribute name="NAME" x="113.284" y="155.321" size="1.778" layer="95"/>
+<attribute name="VALUE" x="113.284" y="150.241" size="1.778" layer="96"/>
+</instance>
 <instance part="FB1" gate="G$1" x="101.6" y="160.02" smashed="yes" rot="R90">
 <attribute name="NAME" x="113.03" y="175.26" size="1.778" layer="95" rot="R180" align="center-left"/>
 <attribute name="VALUE" x="130.81" y="172.72" size="1.778" layer="96" rot="R180" align="center-left"/>
 </instance>
-<instance part="J15" gate="G$1" x="115.57" y="71.12"/>
-<instance part="J16" gate="G$1" x="115.57" y="55.88"/>
-<instance part="J17" gate="G$1" x="115.57" y="95.885"/>
+<instance part="J15" gate="G$1" x="115.57" y="71.12" smashed="yes">
+<attribute name="VALUE" x="114.3" y="63.5" size="1.778" layer="96"/>
+<attribute name="NAME" x="114.3" y="76.962" size="1.778" layer="95"/>
+</instance>
+<instance part="J16" gate="G$1" x="115.57" y="55.88" smashed="yes">
+<attribute name="VALUE" x="114.3" y="48.26" size="1.778" layer="96"/>
+<attribute name="NAME" x="114.3" y="61.722" size="1.778" layer="95"/>
+</instance>
+<instance part="J17" gate="G$1" x="115.57" y="95.885" smashed="yes">
+<attribute name="VALUE" x="114.3" y="88.265" size="1.778" layer="96"/>
+<attribute name="NAME" x="114.3" y="101.727" size="1.778" layer="95"/>
+</instance>
 </instances>
 <busses>
