File: nu_multi/nu_multi_6/nu_multi6_output_board.sch (KiCad schematic (older format))
At the start: 13 parts, among them J1 CONN_01X02, J10 CONN_01X03, J11 CONN_01X02, J12 CONN_01X03, J13 CONN_01X14, J2 CONN_01X03, J3 CONN_01X02, J4 CONN_01X03, J5 CONN_01X02, J6 CONN_01X03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

Commit message: renamed files
Parts:
- J1, J11, J3, J5, J7, J9: symbol Nu-Multi-Board-rescue:CONN_01X02 -> nu_multi6_output_board:CONN_01X02
- J10, J12, J2, J4, J6, J8: symbol Nu-Multi-Board-rescue:CONN_01X03 -> nu_multi6_output_board:CONN_01X03
- J13: symbol Nu-Multi-Board-rescue:CONN_01X14 -> nu_multi6_output_board:CONN_01X14
Changed lines of the file:
@@
 $EndDescr
 $Comp
-L Nu-Multi-Board-rescue:CONN_01X02 J1
+L nu_multi6_output_board:CONN_01X02 J1
 U 1 1 5AA24F79
 P 2050 5220
@@
 $EndComp
 $Comp
-L Nu-Multi-Board-rescue:CONN_01X03 J2
+L nu_multi6_output_board:CONN_01X03 J2
 U 1 1 5AA2537C
 P 2050 5820
@@
 $EndComp
 $Comp
-L Nu-Multi-Board-rescue:CONN_01X02 J3
+L nu_multi6_output_board:CONN_01X02 J3
 U 1 1 5AA25639
 P 2050 3770
@@
 $EndComp
 $Comp
-L Nu-Multi-Board-rescue:CONN_01X03 J4
+L nu_multi6_output_board:CONN_01X03 J4
 U 1 1 5AA2563F
 P 2050 4370
@@
 $EndComp
 $Comp
-L Nu-Multi-Board-rescue:CONN_01X02 J5
+L nu_multi6_output_board:CONN_01X02 J5
 U 1 1 5AA25CA9
 P 2050 2220
@@
 $EndComp
 $Comp
-L Nu-Multi-Board-rescue:CONN_01X03 J6
+L nu_multi6_output_board:CONN_01X03 J6
 U 1 1 5AA25CAF
 P 2050 2820
@@
 $EndComp
 $Comp
-L Nu-Multi-Board-rescue:CONN_01X02 J7
+L nu_multi6_output_board:CONN_01X02 J7
 U 1 1 5AA25CB5
 P 2050 820
@@
 $EndComp
 $Comp
-L Nu-Multi-Board-rescue:CONN_01X03 J8
+L nu_multi6_output_board:CONN_01X03 J8
 U 1 1 5AA25CBB
 P 2050 1420
@@
 $EndComp
 $Comp
-L Nu-Multi-Board-rescue:CONN_01X02 J11
+L nu_multi6_output_board:CONN_01X02 J11
 U 1 1 5AA25DFB
 P 2050 6620
@@
 $EndComp
 $Comp
-L Nu-Multi-Board-rescue:CONN_01X03 J12
+L nu_multi6_output_board:CONN_01X03 J12
 U 1 1 5AA25E01
 P 2050 7220
@@
 $EndComp
 $Comp
-L Nu-Multi-Board-rescue:CONN_01X14 J13
+L nu_multi6_output_board:CONN_01X14 J13
 U 1 1 5AA25EDC
 P 8800 2770
@@
 CH3
 $Comp
-L Nu-Multi-Board-rescue:CONN_01X02 J9
+L nu_multi6_output_board:CONN_01X02 J9
 U 1 1 5AA66B7D
 P 5350 920
@@
 $EndComp
 $Comp
-L Nu-Multi-Board-rescue:CONN_01X03 J10
+L nu_multi6_output_board:CONN_01X03 J10
 U 1 1 5AA66D73
 P 5350 1470
