File: nu_capsule/nu_coil_base/nu_coil_base.kicad_pcb (KiCad board)
At the start: 2 copper layers, 7.9 x 9 mm, 4 parts

Commit message: Removed temporary files
Other:
- net class Default removed

Commit message: updated coil-base
Parts:
- added REF**: Tab, kikit:Tab, F.Cu at (137.9, 97.2)
- added REF**: Tab, kikit:Tab, F.Cu at (133.2, 92.5)
- added REF**: Tab, kikit:Tab, F.Cu at (137.9, 87.8)
- added REF**: Tab, kikit:Tab, F.Cu at (141.7, 92.5)
Changed lines of the file:
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@@
       (net 1 "GND"))
+  )
+  (footprint "kikit:Tab" (layer "F.Cu")
+    (at 137.95 97.25 90)
+    (descr "A symbol representing annotation for tab placement")
+    (attr exclude_from_pos_files exclude_from_bom)
+    (fp_text reference "REF**" (at 0 -2 90) (layer "F.SilkS") hide
+      (effects (font (size 1 1) (thickness 0.15)))
+    )
+    (fp_text value "Tab" (at -2.75 -1 90) (layer "Dwgs.User")
+      (effects (font (size 1.2 1.2) (thickness 0.2)))
+    )
+    (fp_text user "KIKIT: width: 3mm" (at -5.5 0) (layer "Dwgs.User")
+      (effects (font (size 1 1) (thickness 0.15)))
+    )
+    (fp_line (start 0.25 1) (end 0.25 -1) (layer "Dwgs.User") (width 0.3))
+    (fp_line (start 0.25 0) (end -0.75 -1) (layer "Dwgs.User") (width 0.3))
+    (fp_line (start 0.25 0) (end -0.75 1) (layer "Dwgs.User") (width 0.3))
+    (fp_line (start 0.25 0) (end -2.75 0) (layer "Dwgs.User") (width 0.3))
+  )
+  (footprint "kikit:Tab" (layer "F.Cu")
+    (at 133.25 92.5)
+    (descr "A symbol representing annotation for tab placement")
+    (attr exclude_from_pos_files exclude_from_bom)
+    (fp_text reference "REF**" (at 0 -2) (layer "F.SilkS") hide
+      (effects (font (size 1 1) (thickness 0.15)))
+    )
+    (fp_text value "Tab" (at -2.75 -1) (layer "Dwgs.User")
+      (effects (font (size 1.2 1.2) (thickness 0.2)))
+    )
+    (fp_text user "KIKIT: width: 5mm" (at -5.5 0 90) (layer "Dwgs.User")
+      (effects (font (size 1 1) (thickness 0.15)))
+    )
+    (fp_line (start 0.25 1) (end 0.25 -1) (layer "Dwgs.User") (width 0.3))
+    (fp_line (start 0.25 0) (end -0.75 1) (layer "Dwgs.User") (width 0.3))
+    (fp_line (start 0.25 0) (end -0.75 -1) (layer "Dwgs.User") (width 0.3))
+    (fp_line (start 0.25 0) (end -2.75 0) (layer "Dwgs.User") (width 0.3))
+  )
+  (footprint "kikit:Tab" (layer "F.Cu")
+    (at 137.95 87.75 -90)
+    (descr "A symbol representing annotation for tab placement")
+    (attr exclude_from_pos_files exclude_from_bom)
+    (fp_text reference "REF**" (at 0 -2 90) (layer "F.SilkS") hide
+      (effects (font (size 1 1) (thickness 0.15)))
+    )
+    (fp_text value "Tab" (at -2.75 -1 90) (layer "Dwgs.User")
+      (effects (font (size 1.2 1.2) (thickness 0.2)))
+    )
+    (fp_text user "KIKIT: width: 3mm" (at -5.5 0) (layer "Dwgs.User")
+      (effects (font (size 1 1) (thickness 0.15)))
+    )
+    (fp_line (start 0.25 1) (end 0.25 -1) (layer "Dwgs.User") (width 0.3))
+    (fp_line (start 0.25 0) (end -2.75 0) (layer "Dwgs.User") (width 0.3))
+    (fp_line (start 0.25 0) (end -0.75 -1) (layer "Dwgs.User") (width 0.3))
+    (fp_line (start 0.25 0) (end -0.75 1) (layer "Dwgs.User") (width 0.3))
+  )
+  (footprint "kikit:Tab" (layer "F.Cu")
+    (at 141.7 92.5 180)
+    (descr "A symbol representing annotation for tab placement")
+    (attr exclude_from_pos_files exclude_from_bom)
+    (fp_text reference "REF**" (at 0 -2) (layer "F.SilkS") hide
+      (effects (font (size 1 1) (thickness 0.15)))
+    )
+    (fp_text value "Tab" (at -2.75 -1) (layer "Dwgs.User")
+      (effects (font (size 1.2 1.2) (thickness 0.2)))
+    )
+    (fp_text user "KIKIT: width: 5mm" (at -5.5 0 90) (layer "Dwgs.User")
+      (effects (font (size 1 1) (thickness 0.15)))
+    )
+    (fp_line (start 0.25 1) (end 0.25 -1) (layer "Dwgs.User") (width 0.3))
+    (fp_line (start 0.25 0) (end -0.75 -1) (layer "Dwgs.User") (width 0.3))
+    (fp_line (start 0.25 0) (end -2.75 0) (layer "Dwgs.User") (width 0.3))
+    (fp_line (start 0.25 0) (end -0.75 1) (layer "Dwgs.User") (width 0.3))
   )
   (gr_circle (center 137.45 92.5) (end 141.45 92.5) (layer "Dwgs.User") (width 0.1) (fill none))

Commit message: Minimize tabs for fabrication
Parts:
- removed the REF** at (137.9, 97.2)
- removed the REF** at (137.9, 87.8)
Changed lines of the file:
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@@
-  )
-  (footprint "kikit:Tab" (layer "F.Cu")
-    (at 137.95 97.25 90)
-    (descr "A symbol representing annotation for tab placement")
-    (attr exclude_from_pos_files exclude_from_bom)
-    (fp_text reference "REF**" (at 0 -2 90) (layer "F.SilkS") hide
-      (effects (font (size 1 1) (thickness 0.15)))
-    )
-    (fp_text value "Tab" (at -2.75 -1 90) (layer "Dwgs.User")
-      (effects (font (size 1.2 1.2) (thickness 0.2)))
-    )
-    (fp_text user "KIKIT: width: 3mm" (at -5.5 0) (layer "Dwgs.User")
-      (effects (font (size 1 1) (thickness 0.15)))
-    )
-    (fp_line (start 0.25 1) (end 0.25 -1) (layer "Dwgs.User") (width 0.3))
-    (fp_line (start 0.25 0) (end -0.75 -1) (layer "Dwgs.User") (width 0.3))
-    (fp_line (start 0.25 0) (end -0.75 1) (layer "Dwgs.User") (width 0.3))
-    (fp_line (start 0.25 0) (end -2.75 0) (layer "Dwgs.User") (width 0.3))
   )
   (footprint "kikit:Tab" (layer "F.Cu")
@@
   )
   (footprint "kikit:Tab" (layer "F.Cu")
-    (at 137.95 87.75 -90)
-    (descr "A symbol representing annotation for tab placement")
-    (attr exclude_from_pos_files exclude_from_bom)
-    (fp_text reference "REF**" (at 0 -2 90) (layer "F.SilkS") hide
-      (effects (font (size 1 1) (thickness 0.15)))
-    )
-    (fp_text value "Tab" (at -2.75 -1 90) (layer "Dwgs.User")
-      (effects (font (size 1.2 1.2) (thickness 0.2)))
-    )
-    (fp_text user "KIKIT: width: 3mm" (at -5.5 0) (layer "Dwgs.User")
-      (effects (font (size 1 1) (thickness 0.15)))
-    )
-    (fp_line (start 0.25 1) (end 0.25 -1) (layer "Dwgs.User") (width 0.3))
-    (fp_line (start 0.25 0) (end -2.75 0) (layer "Dwgs.User") (width 0.3))
-    (fp_line (start 0.25 0) (end -0.75 -1) (layer "Dwgs.User") (width 0.3))
-    (fp_line (start 0.25 0) (end -0.75 1) (layer "Dwgs.User") (width 0.3))
-  )
-  (footprint "kikit:Tab" (layer "F.Cu")
