File: nu_multi/output_board/nu_multi_output_board.kicad_sch (KiCad schematic)
At the start: 2 parts, among them J1 Conn_02x07_Odd_Even, J2 Conn_02x05_Odd_Even

Commit message: Updated. Use cycfi library.
Parts:
- J1: footprint Pin_Headers:Pin_Header_Straight_2x07_Pitch1.00mm_SMD -> cycfi_library:pin_header_2x7p_1.00mm_smd_vertical
- J2: footprint Cycfi_Kicad_Headers:2x5_1mm_Angled_SMD -> cycfi_library:2x5_2mm_Nu_Multi_SMD
