File: nu_multi/nu_multi_7/nu_multi7_mounting_board.kicad_sch (KiCad schematic)
At the start: 8 parts, among them J15 CONN_01X14, U1 nu_capsule, U2 nu_capsule, U3 nu_capsule, U4 nu_capsule, U5 nu_capsule, U6 nu_capsule, U7 nu_capsule

Commit message: Use 2x7p connector from cycfi lib
Parts:
- J15: footprint Pin_Headers:Pin_Header_Straight_2x07_Pitch1.00mm_SMD -> cycfi_library:pin_header_2x7p_1.00mm_smd_vertical
Changed lines of the file:
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@@
     (property "Reference" "J15" (id 0) (at 195.58 54.61 0))
     (property "Value" "CONN_01X14" (id 1) (at 194.945 93.091 0))
-    (property "Footprint" "Pin_Headers:Pin_Header_Straight_2x07_Pitch1.00mm_SMD" (id 2) (at 195.58 73.66 0)
+    (property "Footprint" "cycfi_library:pin_header_2x7p_1.00mm_smd_vertical" (id 2) (at 195.58 73.66 0)
       (effects (font (size 1.27 1.27)) hide)
     )
@@
     )
     (path "/00000000-0000-0000-0000-00005b39e78d"
-      (reference "J15") (unit 1) (value "CONN_01X14") (footprint "Pin_Headers:Pin_Header_Straight_2x07_Pitch1.00mm_SMD")
+      (reference "J15") (unit 1) (value "CONN_01X14") (footprint "cycfi_library:pin_header_2x7p_1.00mm_smd_vertical")
     )
     (path "/3b032e5e-9eca-44a1-bdcb-8a1f80754daf"
