File: nu_multi/nu_multi_8_10.2mm/nu_multi8_mounting_board.kicad_pcb (KiCad board)
At the start: 2 copper layers, 91.5 x 18 mm, 10 parts, among them J13 CONN_01X14, U1 nu_capsule, U2 nu_capsule, U3 nu_capsule, U4 nu_capsule, U5 nu_capsule, U6 nu_capsule, U7 nu_capsule, U8 nu_capsule

Commit message: - Add fab single - Bump the version. This should have been v2.8.
Other:
- board text added: "Nu Multi 8 v2.8 10.5mm"
- board text removed: "Nu Multi 8 v2.54 10.5mm"
Changed lines of the file:
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@@
 		(layer "Edge.Cuts")
 	)
-	(gr_text "Nu Multi 8 \nv2.54\n10.5mm\n"
+	(gr_text "Nu Multi 8 \nv2.8\n10.5mm\n"
 		(at 179.8 91.07 0)
 		(layer "F.SilkS")
