File: nu_multi/nu_multi_jb4/nu_multi_jb4_mounting_board.kicad_sch (KiCad schematic)
At the start: 5 parts, among them J13 CONN_01X14, U1 nu_capsule, U2 nu_capsule, U3 nu_capsule, U4 nu_capsule

Commit message: Updated PCB mounting board and drawing guide
Other:
- company: Document Number: 2021009 -> Document Number: 2025007
- title: Nu Multi 6 Output Board -> Nu Multi JB4 Output Board
Changed lines of the file:
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@@
 	(paper "A4")
 	(title_block
-		(title "Nu Multi 6 Output Board")
-		(date "2025-03-20")
+		(title "Nu Multi JB4 Output Board")
+		(date "2025-08-23")
 		(rev "v2.54")
-		(company "Document Number: 2021009")
+		(company "Document Number: 2025007")
 	)
 	(text "NC"
@@
 			)
 		)
-		(property "Description" ""
+		(property "Description" "Power symbol creates a global label with name \"GND\" , ground"
 			(at 160.02 48.26 0)
 			(effects
@@
 			)
 		)
-		(property "Description" ""
+		(property "Description" "Power symbol creates a global label with name \"GND\" , ground"
 			(at 177.8 83.82 0)
 			(effects
@@
 	)
 	(symbol
-		(lib_name "nu_capsule_3")
 		(lib_id "cycfi_library:nu_capsule")
 		(at 73.66 53.34 0)
@@
 			)
 		)
-		(property "Description" ""
+		(property "Description" "Special symbol for telling ERC where power comes from"
 			(at 172.72 50.8 0)
 			(effects
@@
 			)
 		)
-		(property "Description" ""
+		(property "Description" "Power symbol creates a global label with name \"GND\" , ground"
 			(at 73.66 128.27 0)
 			(effects
@@
 			)
 		)
-		(property "Description" ""
+		(property "Description" "Power symbol creates a global label with name \"GND\" , ground"
 			(at 73.66 83.82 0)
 			(effects
@@
 	)
 	(symbol
-		(lib_name "nu_capsule_2")
 		(lib_id "cycfi_library:nu_capsule")
 		(at 73.66 99.06 0)
@@
 			)
 		)
-		(property "Description" ""
+		(property "Description" "Power symbol creates a global label with name \"GND\" , ground"
 			(at 73.66 106.68 0)
 			(effects
@@
 	)
 	(symbol
-		(lib_name "nu_capsule_1")
 		(lib_id "cycfi_library:nu_capsule")
 		(at 73.66 120.65 0)
@@
 			)
 		)
-		(property "Description" ""
+		(property "Description" "Special symbol for telling ERC where power comes from"
 			(at 172.72 48.26 0)
 			(effects
@@
 	)
 	(symbol
-		(lib_name "nu_capsule_4")
 		(lib_id "cycfi_library:nu_capsule")
 		(at 73.66 76.2 0)
@@
 			)
 		)
-		(property "Description" ""
+		(property "Description" "Power symbol creates a global label with name \"GND\" , ground"
 			(at 73.66 60.96 0)
 			(effects
